File: CarCANdy-PCB/CarCANdy-PCB.kicad_sch (KiCad schematic)
At the start: 2 parts, among them U1 Teensy4.1, U2 ESP32-C3_SUPERMINI_TH

Commit message: implemented filtering (untested), added tmux build script, started PCB
Parts:
- added U3: SN65HVD233DR, SN65HVD233DR:SOIC127P599X175-8N, symbol SN65HVD233DR:SN65HVD233DR
Connections:
- net +3.3V: now also U3.3 (VCC)
- net GND: now also U3.2 (GND)
- net CAN2_TX: now reaches U1.2 (0_RX1_CRX2_CS1)
- net CAN3_RX: now reaches U1.22 (30_CRX3)
- net CAN3_TX: now reaches U1.23 (31_CTX3)
- net CAN2_RX: now reaches U1.3 (1_TX1_CTX2_MISO1)
- net CAN1_TX: now reaches U1.44 (22_A8_CTX1)
- net CAN1_RX: now reaches U1.45 (23_A9_CRX1_MCLK1)
- net CAN1_RX: now also U3.4 (RXD)
- new net CAN1_H: U3.7 (CANH)
- new net CAN1_L: U3.6 (CANL)
Other:
- moved on the sheet: U1, U2

Commit message: added to PCB
Parts:
- removed U1: Teensy4.1, Teensy:Teensy41, symbol Teensy:Teensy4.1
- added ADC1, ADC2, RS1, RS2, RS3: RS, Jumper:SolderJumper-2_P1.3mm_Open_TrianglePad1.0x1.5mm, symbol Jumper:SolderJumper_2_Open
- added C1, C2: 100nF, Capacitor_SMD:C_0603_1608Metric_Pad1.08x0.95mm_HandSolder, symbol Device:C
- added D1, D2, D3: NUP2105LT1G, nup2105lt1g:SOT95P237X111-3N, symbol nup2105lt1g:NUP2105LT1G
- added D4: SS14, Diode_SMD:D_SMA, symbol Diode:SS14
- added D5: 1N4148W, Diode_SMD:D_SOD-123, symbol Diode:1N4148W
- added D6, D7: BAT54S, Package_TO_SOT_SMD:SOT-23, symbol Diode:BAT54S
- added J1: 8P8C_Shielded, Connector_RJ:RJ45_RCH_RC01937, symbol Connector:8P8C_Shielded
- added J2: Power, Connector_JST:JST_EH_S3B-EH_1x03_P2.50mm_Horizontal, symbol Connector:Conn_01x03_Pin
- added JP2, JP6, JP9: RS, Connector_PinHeader_2.54mm:PinHeader_1x03_P2.54mm_Vertical, symbol Jumper:Jumper_3_Open
- added K1: IM06TS, IM06:RELAY_IM06TS, symbol IM06:IM06TS
- added PSU1: 12v-5v_mini_buck, Library:mini12v-5v_buck, symbol Connector:Conn_01x04_Pin
- added Q2: BC847C, Package_TO_SOT_SMD:SOT-23, symbol Transistor_BJT:BC847
- added Q3: AO3407A, Package_TO_SOT_SMD:SOT-23, symbol Transistor_FET:AO3401A
- added R1, R3, R5: 120, Resistor_SMD:R_0603_1608Metric_Pad0.98x0.95mm_HandSolder, symbol Device:R_US
- added R10, R14: 33K, Resistor_SMD:R_0603_1608Metric_Pad0.98x0.95mm_HandSolder, symbol Device:R_US
- added R11: 100, Resistor_SMD:R_0603_1608Metric_Pad0.98x0.95mm_HandSolder, symbol Device:R_US
- added R12, R15, R18: 47k, Resistor_SMD:R_0603_1608Metric_Pad0.98x0.95mm_HandSolder, symbol Device:R_US
- added R13: 22K, Resistor_SMD:R_0603_1608Metric_Pad0.98x0.95mm_HandSolder, symbol Device:R_US
- added R16: 15K, Resistor_SMD:R_0603_1608Metric_Pad0.98x0.95mm_HandSolder, symbol Device:R_US
- added R17: 4.7K, Resistor_SMD:R_0603_1608Metric_Pad0.98x0.95mm_HandSolder, symbol Device:R_US
- added R2, R4, R6: 10K, Resistor_SMD:R_0603_1608Metric_Pad0.98x0.95mm_HandSolder, symbol Device:R_US
- added R7: 2.2K, Resistor_SMD:R_0603_1608Metric_Pad0.98x0.95mm_HandSolder, symbol Device:R_US
- added R8: 10k, Resistor_SMD:R_0603_1608Metric_Pad0.98x0.95mm_HandSolder, symbol Device:R_US
- added R9: 180K, Resistor_SMD:R_0603_1608Metric_Pad0.98x0.95mm_HandSolder, symbol Device:R_US
- added T1: NTD5867NL, NTD5867NL:DPACK, symbol NTD5867NL:NTD5867NL
- added TERM1, TERM2, TERM3: TERM, Jumper:SolderJumper-2_P1.3mm_Open_TrianglePad1.0x1.5mm, symbol Jumper:SolderJumper_2_Open
- added U4, U5: SN65HVD233DR, SN65HVD233DR:SOIC127P599X175-8N, symbol SN65HVD233DR:SN65HVD233DR
- added U6: Teensy4.1, Teensy:Teensy41, symbol Teensy:Teensy4.1
- added U7: LTV-817S, Package_DIP:SMDIP-4_W9.53mm, symbol Isolator:LTV-817S
Connections:
- net +3.3V: now also D6.2 (K), D7.2 (K), JP2.3 (B), JP6.3 (B), JP9.3 (B), R8.2, U4.3 (VCC), U5.3 (VCC), U6.46 (3V3)
- net +5V: now also PSU1.5v+ (Pin_4), U6.48 (VIN)
- net CAN1_H: now also D1.2, J1.7, TERM1.2 (B)
- net CAN1_L: now also D1.1, J1.8, R1.2
- net CAN1_RX: now also U6.45 (23_A9_CRX1_MCLK1)
- net CAN1_TX: now also U3.1 (TXD), U6.44 (22_A8_CTX1)
- net CAN2_RX: now also U4.4 (RXD), U6.3 (1_TX1_CTX2_MISO1)
- net CAN2_TX: now also U4.1 (TXD), U6.2 (0_RX1_CRX2_CS1)
- net CAN3_RX: now also U5.4 (RXD), U6.22 (30_CRX3)
- net CAN3_TX: now also U5.1 (TXD), U6.23 (31_CTX3)
- net GND: now also C1.2, C2.2, D1.3, D2.3, D3.3, D5.2 (A), D6.1 (A), D7.1 (A), J1.3, J1.SH, J2.3 (Pin_3), K1.8, PSU1.12v- (Pin_2), PSU1.5v- (Pin_3), Q2.2 (E), R10.2, R12.2, R14.2, R18.2, R2.1, R4.1, R6.1, RS1.2 (B), RS2.2 (B), RS3.2 (B), T1.3, U4.2 (GND), U5.2 (GND), U6.58 (GND), U6.59 (GND), U7.2, U7.3
- net T_RX->E_TX: now also U6.9 (7_RX2_OUT1A)
- net T_TX->E_RX: now also U6.10 (8_TX2_IN1)
- net at U3.8 (RS): now also JP2.2 (C)
- new net: ADC1.1 (A), R9.1
- new net: R3.1, TERM2.1 (A)
- new net: ADC2.1 (A), R13.1
- new net: JP6.1 (A), R4.2, RS2.1 (A)
- new net: JP9.1 (A), R6.2, RS3.1 (A)
- new net: R11.2, R12.1, T1.1
- new net: JP9.2 (C), U5.8 (RS)
- new net: JP2.1 (A), R2.2, RS1.1 (A)
- new net: R1.1, TERM1.1 (A)
- new net: Q3.1 (G), R15.2, R16.1
- new net: JP6.2 (C), U4.8 (RS)
- new net: Q2.1 (B), R17.2
- new net: Q2.3 (C), R16.2
- new net: R5.1, TERM3.1 (A)
- new net: D5.1 (K), R7.2, U7.1
- new net +12V: D4.1 (K), K1.4, PSU1.12v+ (Pin_1), Q3.3 (D), R15.1
- new net 12V_INPUT: R7.1
- new net 12V_SIG: ADC1.2 (B), ADC2.2 (B)
- new net 12v_CONST: J2.1 (Pin_1), K1.3
- new net 12v_IGN: J2.2 (Pin_2), K1.1
- new net 12v_OUT: Q3.2 (S)
- new net ADC: C1.1, C2.1, D6.3 (COM), D7.3 (COM), R10.1, R13.2, R14.1, R9.2
- new net CAN2_H: D2.2, J1.6, TERM2.2 (B), U4.7 (CANH)
- new net CAN2_L: D2.1, J1.4, R3.2, U4.6 (CANL)
- new net CAN3_H: D3.2, J1.2, TERM3.2 (B), U5.7 (CANH)
- new net CAN3_L: D3.1, J1.1, R5.2, U5.6 (CANL)
- new net GPIO: R11.1, R17.1, R18.1, R8.1, U7.4
- new net OUT_LOW: D4.2 (A), T1.2
Other:
- note added: "12V ADC"
- note added: "12V Active High Input"
- note added: "12V Active Low Output"
- note added: "12v in = GPIO LOW"
- note added: "5V ADC"
- note added: "CAN"
- note added: "CAN1"
- note added: "CAN2"
- note added: "GPIO HIGH = 12+"
- note added: "GPIO HIGH = path to ground"
- note added: "Power"
- moved on the sheet: U3

Commit message: added to PCB
Parts:
- removed ADC1, ADC2: RS, Jumper:SolderJumper-2_P1.3mm_Open_TrianglePad1.0x1.5mm, symbol Jumper:SolderJumper_2_Open
- removed C1: 100nF, Capacitor_SMD:C_0603_1608Metric_Pad1.08x0.95mm_HandSolder, symbol Device:C
- removed D4: SS14, Diode_SMD:D_SMA, symbol Diode:SS14
- removed D6: BAT54S, Package_TO_SOT_SMD:SOT-23, symbol Diode:BAT54S
- removed J2: Power, Connector_JST:JST_EH_S3B-EH_1x03_P2.50mm_Horizontal, symbol Connector:Conn_01x03_Pin
- removed K1: IM06TS, IM06:RELAY_IM06TS, symbol IM06:IM06TS
- removed Q2: BC847C, Package_TO_SOT_SMD:SOT-23, symbol Transistor_BJT:BC847
- removed Q3: AO3407A, Package_TO_SOT_SMD:SOT-23, symbol Transistor_FET:AO3401A
- removed R10: 33K, Resistor_SMD:R_0603_1608Metric_Pad0.98x0.95mm_HandSolder, symbol Device:R_US
- removed R11: 100, Resistor_SMD:R_0603_1608Metric_Pad0.98x0.95mm_HandSolder, symbol Device:R_US
- removed R12: 47k, Resistor_SMD:R_0603_1608Metric_Pad0.98x0.95mm_HandSolder, symbol Device:R_US
- removed R9: 180K, Resistor_SMD:R_0603_1608Metric_Pad0.98x0.95mm_HandSolder, symbol Device:R_US
- removed T1: NTD5867NL, NTD5867NL:DPACK, symbol NTD5867NL:NTD5867NL
- removed U7: LTV-817S, Package_DIP:SMDIP-4_W9.53mm, symbol Isolator:LTV-817S
- added C3, C4, C5, C6, C7: 100nF, Capacitor_SMD:C_0603_1608Metric_Pad1.08x0.95mm_HandSolder, symbol Device:C
- added D10, D11, D12, D8, D9: 1N4148W, Diode_SMD:D_SOD-123, symbol Diode:1N4148W
- added D13, D14: BAT54S, Package_TO_SOT_SMD:SOT-23, symbol Diode:BAT54S
- added J2: Power, Connector_JST:JST_EH_S2B-EH_1x02_P2.50mm_Horizontal, symbol Connector:Conn_01x02_Pin
- added J3, J5, J6, J7, J9: TB004-508-03BE, TB004-508-03BE:CUI_TB004-508-03BE, symbol TB004-508-03BE:TB004-508-03BE
- added J4, J8: AUART1, Connector_JST:JST_PH_S4B-PH-K_1x04_P2.00mm_Horizontal, symbol Connector:Conn_01x04_Pin
- added K3, K4, K5: IM02, IM06:RELAY_IM06TS, symbol Relay:IM02
- added Q1, Q2, Q3: AO3400A, Package_TO_SOT_SMD:SOT-23, symbol Transistor_FET:AO3400A
- added R19, R25, R27: 100, Resistor_SMD:R_0603_1608Metric_Pad0.98x0.95mm_HandSolder, symbol Device:R_US
- added R20, R26, R28: 47K, Resistor_SMD:R_0603_1608Metric_Pad0.98x0.95mm_HandSolder, symbol Device:R_US
- added R21, R23: 2.2K, Resistor_SMD:R_0603_1608Metric_Pad0.98x0.95mm_HandSolder, symbol Device:R_US
- added R22, R24: 10k, Resistor_SMD:R_0603_1608Metric_Pad0.98x0.95mm_HandSolder, symbol Device:R_US
- added SW2, SW3, SW4: JS202011CQN, JS202011CQN:JS202011CQN, symbol Switch:SW_DPDT_x2
- added U1, U7, U8: LTV-357T, Package_SO:SO-4_4.4x3.6mm_P2.54mm, symbol Isolator:LTV-357T
- R15: value 47k -> 22K
- R16: value 15K -> 33K
- R17: value 4.7K -> 22K
- R18: value 47k -> 33K
Connections:
- net ADC is gone; now on net ADC1: C2.1, D7.3 (COM), R13.2, R14.1
- net +12V: now also J2.1 (Pin_1), SW2.1 (A), SW3.1 (A), SW4.1 (A); no longer R15.1
- net +3.3V: now also D13.2 (K), D14.2 (K), R22.2, R24.2
- net +5V: now also C3.1, C4.1, C5.1, D11.1 (K), D12.1 (K), D8.1 (K), J4.1 (Pin_1), J8.1 (Pin_1), K3.1, K4.1, K5.1
- net GND: now also R16.2, U6.1 (GND), U6.34 (GND), U6.47 (GND), U6.52 (GND), C6.2, C7.2, D13.1 (A), D14.1 (A), J2.2 (Pin_2), J4.4 (Pin_4), J8.4 (Pin_4), Q1.2 (S), Q2.2 (S), Q3.2 (S), R20.2, R26.2, R28.2, SW2.6 (C), SW3.6 (C), SW4.6 (C), U1.3, U7.3, U8.3; no longer D5.2 (A)
- net 5V_SIG1: now reaches R13.1
- net 5V_SIG1: now also J9.1
- net ADC2: now reaches R15.2, R16.1
- net ADC2: now also U6.36 (14_A0_TX3_SPDIF_OUT), C6.1, D13.3 (COM)
- net ADC3: now reaches R17.2
- net ADC3: now also R18.1, U6.33 (41_A17), C7.1, D14.3 (COM)
- net at D5.1 (K), R7.2: now also U1.1
- net GPIO_OUT1: now reaches U6.14 (12_MISO_MQSL)
- net GPIO_OUT1: now also R19.1, R20.1
- net ATX2: now reaches U6.16 (24_A10_TX6_SCL2)
- net ATX2: now also J8.3 (Pin_3)
- net ARX2: now reaches U6.17 (25_A11_RX6_SDA2)
- net ARX2: now also J8.2 (Pin_2)
- net GPIO_OUT2: now reaches U6.18 (26_A12_MOSI1)
- net GPIO_OUT2: now also R25.1, R26.1
- net GPIO_OUT3: now reaches U6.19 (27_A13_SCK1)
- net GPIO_OUT3: now also R27.1, R28.1
- net ARX1: now reaches U6.20 (28_RX7)
- net ARX1: now also J4.2 (Pin_2)
- net ATX1: now reaches U6.21 (29_TX7)
- net ATX1: now also J4.3 (Pin_3)
- net ADC1: now reaches U6.37 (15_A1_RX3_SPDIF_IN)
- net GPIO_IN1: now reaches U6.4 (2_OUT2)
- net GPIO_IN1: now also R8.1, U1.4
- net GPIO_IN2: now reaches U6.5 (3_LRCLK2)
- net GPIO_IN2: now also R22.1, U7.4
- net GPIO_IN3: now reaches U6.6 (4_BCLK2)
- net GPIO_IN3: now also R24.1, U8.4
- net 12V_INPUT: no longer names the net of R7.1
- net 12V_INPUT: now also SW2.2 (B)
- removed net GPIO: R17.1, R18.1, R8.1
- new net: D5.2 (A), SW2.5 (B), U1.2
- new net: Q2.1 (G), R25.2
- new net: C4.2, D11.2 (A), K4.8, Q2.3 (D)
- new net: R23.1, SW4.2 (B)
- new net: D10.1 (K), R23.2, U8.1
- new net: D10.2 (A), SW4.5 (B), U8.2
- new net: C3.2, D8.2 (A), K3.8, Q1.3 (D)
- new net: J5.3, K4.5
- new net: J5.2, K4.6
- new net: J5.1, K4.7
- new net: J7.3, K3.5
- new net: J7.2, K3.6
- new net: J7.1, K3.7
- new net: Q3.1 (G), R27.2
- new net: R21.1, SW3.2 (B)
- new net: D9.1 (K), R21.2, U7.1
- new net: C5.2, D12.2 (A), K5.8, Q3.3 (D)
- new net: Q1.1 (G), R19.2
- new net: J6.3, K5.5
- new net: J6.2, K5.6
- new net: J6.1, K5.7
- new net: D9.2 (A), SW3.5 (B), U7.2
- new net 12V_SELECT_INPUT1: J3.1, SW2.3 (C), SW2.4 (A)
- new net 12V_SELECT_INPUT2: J3.2, SW3.3 (C), SW3.4 (A)
- new net 12V_SELECT_INPUT3: J3.3, SW4.3 (C), SW4.4 (A)
- new net 5V_SIG2: J9.2, R15.1
- new net 5V_SIG3: J9.3, R17.1
Other:
- note added: "12V Relay Output"
- note added: "12V Selectable Input"
- note added: "AUX UART"
- note removed: "12V ADC"
- note removed: "12V Active High Input"
- note removed: "12V Active Low Output"
- note removed: "12v in = GPIO LOW"
- note removed: "GPIO HIGH = 12+"
- note removed: "GPIO HIGH = path to ground"
- moved on the sheet: C2, D7, R13, R14, R7, R8

Commit message: added to PCB
Connections:
- net CAN1_H: now also D1.1; no longer D1.2
- net CAN1_L: now also D1.2; no longer D1.1
Changed lines of the file:
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@@
 		)
 	)
-	(global_label "CAN1_L"
+	(global_label "CAN1_H"
 		(shape input)
 		(at 511.81 107.95 180)
@@
 		)
 		(property "Intersheetrefs" "${INTERSHEET_REFS}"
-			(at 501.9305 107.95 0)
+			(at 501.6281 107.95 0)
 			(show_name no)
 			(do_not_autoplace no)
@@
 		)
 	)
-	(global_label "CAN1_H"
+	(global_label "CAN1_L"
 		(shape input)
 		(at 511.81 113.03 180)
@@
 		)
 		(property "Intersheetrefs" "${INTERSHEET_REFS}"
-			(at 501.6281 113.03 0)
+			(at 501.9305 113.03 0)
 			(show_name no)
 			(do_not_autoplace no)

Commit message: added to PCB
Parts:
- added J10, J11: ADC1, Connector_JST:JST_XH_S3B-XH-A-1_1x03_P2.50mm_Horizontal, symbol Connector:Conn_01x03_Pin
- added J12: ADC1, Connector_JST:JST_EH_S3B-EH_1x03_P2.50mm_Horizontal, symbol Connector:Conn_01x03_Pin
- added J13, J14, J15: Conn_01x02_Pin, Connector_JST:JST_XH_S2B-XH-A-1_1x02_P2.50mm_Horizontal, symbol Connector:Conn_01x02_Pin
- added JP1, JP3, JP4: VSEL, Connector_PinHeader_2.00mm:PinHeader_1x03_P2.00mm_Vertical, symbol Jumper:Jumper_3_Open
- C7, D14, J3, J9, R17, R18: now not fitted; now left out of the parts list
- D1, D2, D3: footprint nup2105lt1g:SOT95P237X111-3N -> Package_TO_SOT_SMD:SOT-23-3
- J2: footprint Connector_JST:JST_EH_S2B-EH_1x02_P2.50mm_Horizontal -> Connector_JST:JST_VH_S2P-VH_1x02_P3.96mm_Horizontal
- J4, J8: footprint Connector_JST:JST_PH_S4B-PH-K_1x04_P2.00mm_Horizontal -> Connector_JST:JST_XH_S4B-XH-A-1_1x04_P2.50mm_Horizontal
- J5, J6, J7: value TB004-508-03BE -> JSTVH3; footprint TB004-508-03BE:CUI_TB004-508-03BE -> Connector_JST:JST_VH_S3P-VH_1x03_P3.96mm_Horizontal
- U1, U7, U8: footprint Package_SO:SO-4_4.4x3.6mm_P2.54mm -> Package_SO:SOP-4_3.8x4.1mm_P2.54mm
Connections:
- net +12V: now also JP1.1 (A), JP3.1 (A), JP4.1 (A)
- net +5V: now also J10.1 (Pin_1), J11.1 (Pin_1), J12.1 (Pin_1)
- net 12V_SELECT_INPUT1: now also J13.1 (Pin_1)
- net 12V_SELECT_INPUT2: now also J14.1 (Pin_1)
- net 12V_SELECT_INPUT3: now also J15.1 (Pin_1)
- net 5V_SIG1: now also J10.2 (Pin_2)
- net 5V_SIG2: now also J11.2 (Pin_2)
- net 5V_SIG3: now also J12.2 (Pin_2)
- net CAN1_H: now also D1.2; no longer D1.1
- net CAN1_L: now also D1.1; no longer D1.2
- net GND: now also J10.3 (Pin_3), J11.3 (Pin_3), J12.3 (Pin_3), JP1.3 (B), JP3.3 (B), JP4.3 (B)
- new net: J13.2 (Pin_2), JP1.2 (C)
- new net: J15.2 (Pin_2), JP4.2 (C)
- new net: J14.2 (Pin_2), JP3.2 (C)
Other:
- note added: "ESP32/WiFi"
- moved on the sheet: C2, C6, D13, D7, J4, J8, R13, R14, R15, R16, U2

Commit message: added to PCB
Parts:
- removed J3, J9: TB004-508-03BE, TB004-508-03BE:CUI_TB004-508-03BE, symbol TB004-508-03BE:TB004-508-03BE
- JP2, JP6, JP9: footprint Connector_PinHeader_2.54mm:PinHeader_1x03_P2.54mm_Vertical -> Connector_PinHeader_2.00mm:PinHeader_1x03_P2.00mm_Vertical
Other:
- moved on the sheet: C2, C3, C4, C5, C6, C7, D10, D11, D12, D13, D14, D5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
