File: CarCANdy-PCB/CarCANdy-PCB.kicad_pcb (KiCad board)
At the start: 2 copper layers, 110 x 68 mm, 82 parts, among them J1 8P8C_Shielded, J10 ADC1, J11 ADC1, J13 Conn_01x02_Pin, J14 Conn_01x02_Pin, J15 Conn_01x02_Pin, J2 Power, J4 AUART1, J5 JSTVH3, J6 JSTVH3, J7 JSTVH3, J8 AUART1, K3 IM02, K4 IM02, K5 IM02, Q1 AO3400A, Q2 AO3400A, Q3 AO3400A, SW2 JS202011CQN, SW3 JS202011CQN, SW4 JS202011CQN, U1 LTV-357T, U2 ESP32-C3_SUPERMINI_TH, U3 SN65HVD233DR, U4 SN65HVD233DR, U5 SN65HVD233DR, U6 Teensy4.1, U7 LTV-357T, U8 LTV-357T

Commit message: simplified CANDB json
Other:
- board text added: "TODO V2: - rewire RJ45 so pairs are together and in sequence"
Changed lines of the file:
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@@
 		)
 	)
+	(gr_text "TODO V2: \n - rewire RJ45 so pairs are together and in sequence\n"
+		(at 11.597822 -45.040877 0)
+		(layer "Eco1.User")
+		(effects
+			(font
+				(size 1.5 1.5)
+				(thickness 0.3)
+				(bold yes)
+			)
+			(justify left bottom)
+		)
+	)
 	(segment
 		(start -14.061916 -25.830877)
@@
 	)
 	(segment
+		(start -49.772178 -26.080877)
+		(end -48.539416 -26.080877)
+		(width 0.5)
+		(layer "F.Cu")
+		(net "Net-(J13-Pin_2)")
+	)
+	(segment
+		(start -45.759416 -23.300877)
+		(end -39.002178 -23.300877)
+		(width 0.5)
+		(layer "F.Cu")
+		(net "Net-(J13-Pin_2)")
+	)
+	(segment
+		(start -48.539416 -26.080877)
+		(end -45.759416 -23.300877)
+		(width 0.5)
+		(layer "F.Cu")
+		(net "Net-(J13-Pin_2)")
+	)
+	(segment
+		(start -38.519768 -23.783287)
+		(end -38.519768 -25.341229)
+		(width 0.5)
+		(layer "F.Cu")
+		(net "Net-(J13-Pin_2)")
+	)
+	(segment
+		(start -39.002178 -23.300877)
+		(end -38.519768 -23.783287)
+		(width 0.5)
+		(layer "F.Cu")
+		(net "Net-(J13-Pin_2)")
+	)
+	(segment
 		(start 25.712822 -8.924979)
 		(end 25.917822 -9.129979)
@@
 	)
 	(segment
+		(start -49.772178 -17.580877)
+		(end -48.222178 -16.030877)
+		(width 0.5)
+		(layer "F.Cu")
+		(net "Net-(J14-Pin_2)")
+	)
+	(segment
+		(start -38.899768 -16.653287)
+		(end -38.899768 -18.141229)
+		(width 0.5)
+		(layer "F.Cu")
+		(net "Net-(J14-Pin_2)")
+	)
+	(segment
+		(start -48.222178 -16.030877)
+		(end -39.522178 -16.030877)
+		(width 0.5)
+		(layer "F.Cu")
+		(net "Net-(J14-Pin_2)")
+	)
+	(segment
+		(start -39.522178 -16.030877)
+		(end -38.899768 -16.653287)
+		(width 0.5)
+		(layer "F.Cu")
+		(net "Net-(J14-Pin_2)")
+	)
+	(segment
 		(start -20.039768 -11.511229)
 		(end -18.152178 -13.398819)
@@
 	)
 	(segment
+		(start -38.839768 -8.963287)
+		(end -38.839768 -10.401229)
+		(width 0.5)
+		(layer "F.Cu")
+		(net "Net-(J15-Pin_2)")
+	)
+	(segment
+		(start -39.822178 -7.980877)
+		(end -38.839768 -8.963287)
+		(width 0.5)
+		(layer "F.Cu")
+		(net "Net-(J15-Pin_2)")
+	)
+	(segment
+		(start -49.772178 -9.081229)
+		(end -48.671826 -7.980877)
+		(width 0.5)
+		(layer "F.Cu")
+		(net "Net-(J15-Pin_2)")
+	)
+	(segment
+		(start -48.671826 -7.980877)
+		(end -39.822178 -7.980877)
+		(width 0.5)
+		(layer "F.Cu")
+		(net "Net-(J15-Pin_2)")
+	)
+	(segment
 		(start -33.572178 -4.320877)
 		(end -33.302178 -4.050877)
@@
 		(net "Net-(JP6-C)")
 	)
-	(segment
-		(start -49.772178 -26.080877)
-		(end -48.539416 -26.080877)
-		(width 0.5)
-		(layer "F.Cu")
-		(net "Net-(J13-Pin_2)")
-	)
-	(segment
-		(start -45.759416 -23.300877)
-		(end -39.002178 -23.300877)
-		(width 0.5)
-		(layer "F.Cu")
-		(net "Net-(J13-Pin_2)")
-	)
-	(segment
-		(start -48.539416 -26.080877)
-		(end -45.759416 -23.300877)
-		(width 0.5)
-		(layer "F.Cu")
-		(net "Net-(J13-Pin_2)")
-	)
-	(segment
-		(start -38.519768 -23.783287)
-		(end -38.519768 -25.341229)
-		(width 0.5)
-		(layer "F.Cu")
-		(net "Net-(J13-Pin_2)")
-	)
-	(segment
-		(start -39.002178 -23.300877)
-		(end -38.519768 -23.783287)
-		(width 0.5)
-		(layer "F.Cu")
-		(net "Net-(J13-Pin_2)")
-	)
-	(segment
-		(start -49.772178 -17.580877)
-		(end -48.222178 -16.030877)
-		(width 0.5)
-		(layer "F.Cu")
-		(net "Net-(J14-Pin_2)")
-	)
-	(segment
-		(start -38.899768 -16.653287)
-		(end -38.899768 -18.141229)
-		(width 0.5)
-		(layer "F.Cu")
-		(net "Net-(J14-Pin_2)")
-	)
-	(segment
-		(start -48.222178 -16.030877)
-		(end -39.522178 -16.030877)
-		(width 0.5)
-		(layer "F.Cu")
-		(net "Net-(J14-Pin_2)")
-	)
-	(segment
-		(start -39.522178 -16.030877)
-		(end -38.899768 -16.653287)
-		(width 0.5)
-		(layer "F.Cu")
-		(net "Net-(J14-Pin_2)")
-	)
-	(segment
-		(start -38.839768 -8.963287)
-		(end -38.839768 -10.401229)
-		(width 0.5)
-		(layer "F.Cu")
-		(net "Net-(J15-Pin_2)")
-	)
-	(segment
-		(start -39.822178 -7.980877)
-		(end -38.839768 -8.963287)
-		(width 0.5)
-		(layer "F.Cu")
-		(net "Net-(J15-Pin_2)")
-	)
-	(segment
-		(start -49.772178 -9.081229)
-		(end -48.671826 -7.980877)
-		(width 0.5)
-		(layer "F.Cu")
-		(net "Net-(J15-Pin_2)")
-	)
-	(segment
-		(start -48.671826 -7.980877)
-		(end -39.822178 -7.980877)
-		(width 0.5)
-		(layer "F.Cu")
-		(net "Net-(J15-Pin_2)")
-	)
 	(zone

Commit message: simplified CANDB json
Parts:
- added SW1: REBOOT, Button_Switch_SMD:SW_Push_1P1T_NO_CK_KMR2, F.Cu at (76.2, 0.68)
Connections:
- U6 pad 25: unconnected-(U6-33_MCLK2-Pad25) -> Net-(U6-33_MCLK2)
Routing:
- net GND: track 3.62 -> 12.6 mm, vias 12 -> 11
- net T_TX->E_RX: track 77.6 -> 82.6 mm
- net T_RX->E_TX: track 77.7 -> 82.7 mm
- net +5V: track 236.5 -> 232.3 mm
Other:
- board text added: "Note: copper pour under the ESP32 antenna caused WiFi issues"
