File: CarCANdy-PCB/CarCANdy-PCB.kicad_pcb (KiCad board)
At the start: 2 copper layers, 110 x 68 mm, 83 parts, among them J1 8P8C_Shielded, J10 ADC1, J11 ADC1, J13 Conn_01x02_Pin, J14 Conn_01x02_Pin, J15 Conn_01x02_Pin, J2 Power, J4 AUART1, J5 JSTVH3, J6 JSTVH3, J7 JSTVH3, J8 AUART1, K3 IM02, K4 IM02, K5 IM02, Q1 AO3400A, Q2 AO3400A, Q3 AO3400A, SW1 REBOOT, SW2 JS202011CQN, SW3 JS202011CQN, SW4 JS202011CQN, U1 LTV-357T, U2 ESP32-C3_SUPERMINI_TH, U3 SN65HVD233DR, U4 SN65HVD233DR, U5 SN65HVD233DR, U6 Teensy4.1, U7 LTV-357T, U8 LTV-357T

Commit message: bug fixes in PCB
Parts:
- removed SW1: REBOOT, Button_Switch_SMD:SW_Push_1P1T_NO_CK_KMR2
- added D15: 1N4148W, Diode_SMD:D_SOD-123, F.Cu at (10.3, -27.6)
- added D16: 1N4148W, Diode_SMD:D_SOD-123, F.Cu at (33.6, 29.8)
Connections:
- U2 pad 5V: +5V -> Net-(D16-K)
- U6 pad 2: CAN2_TX -> CAN2_RX
- U6 pad 3: CAN2_RX -> CAN2_TX
- U6 pad 48: +5V -> Net-(D15-K)
Routing:
- net GND: track 12.6 -> 3.62 mm
- net CAN2_TX: track 25.0 -> 30.9 mm
- net CAN2_RX: track 28.0 -> 33.4 mm
- net Net-(D15-K): track 0.00 -> 4.76 mm
- net Net-(D16-K): track 0.00 -> 3.48 mm
- net +5V: track 232.3 -> 231.3 mm, vias 0 -> 2

Commit message: added diodes to power rails, rewired RJ45
Parts:
- added SW1: REBOOT, Button_Switch_SMD:SW_Push_1P1T_NO_CK_KMR2, F.Cu at (31.7, -27.1)
Connections:
- J1 pad 1: CAN3_L -> unconnected-(J1-Pad1)
- J1 pad 2: CAN3_H -> GND
- J1 pad 3: GND -> CAN3_H
- J1 pad 4: CAN2_L -> CAN3_L
- J1 pad 5: unconnected-(J1-Pad5) -> CAN2_H
- J1 pad 6: CAN2_H -> CAN2_L
Routing:
- net CAN3_H: track 34.6 -> 42.6 mm
- net CAN2_H: track 31.0 -> 35.5 mm
- net CAN3_L: track 42.5 -> 45.7 mm
- net CAN2_L: track 31.9 -> 34.4 mm
